Commit message: fix: stabilize mapping launch and rviz setup

File: urdf/diff_wheeled_robot_with_laser.xacro (robot description, xacro)
@@ -36,5 +36,5 @@
   <xacro:property name="caster_b_mass" value="0.5" /> <!-- in kg-->
   <!-- Wheels -->
-  <xacro:property name="wheel_mass" value="2.5" /> --> <!-- in kg-->
+  <xacro:property name="wheel_mass" value="2.5" /> <!-- in kg-->
   <xacro:property name="base_x_origin_to_wheel_origin" value="0.25" />
   <xacro:property name="base_y_origin_to_wheel_origin" value="0.3" />
